File: _autosave-GPIO2HUB75.kicad_sch (KiCad schematic)
At the start: 8 parts, among them M1 Noctua

Commit message: version 5
Parts:
- renumbered RPiGPIO to RPiGPIO1
Changed lines of the file:
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@@
   (symbol (lib_id "Connector_Generic:Conn_02x20_Odd_Even") (at 185.42 78.74 0) (unit 1)
     (in_bom yes) (on_board yes) (dnp no)
-    (property "Reference" "RPiGPIO" (at 186.69 52.07 0)
+    (property "Reference" "RPiGPIO1" (at 186.69 52.07 0)
       (effects (font (size 1.27 1.27)))
     )
@@
       (project "GPIO2HUB75"
         (path "/1420b1a7-2230-482f-814a-7ef4eb1c7dc0"
-          (reference "RPiGPIO") (unit 1)
+          (reference "RPiGPIO1") (unit 1)
         )
       )
