File: passive/RP4Passive.kicad_sch (KiCad schematic)
At the start: 8 parts, among them M1 Noctua

Commit message: add back 3.3v for the future co2 sensor
Parts:
- GPIO1: value 02x04 -> 02x05; footprint Connector_PinHeader_2.54mm:PinHeader_2x04_P2.54mm_Horizontal -> Connector_PinHeader_2.54mm:PinHeader_2x05_P2.54mm_Horizontal; symbol Connector_Generic:Conn_02x04_Odd_Even -> Connector_Generic:Conn_02x05_Odd_Even
Connections:
- net at BZ1.2 (+), HUB1.14 (Pin_14), HUB1.4 (Pin_4)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: now also GPIO1.10 (Pin_10), GPIO1.9 (Pin_9); no longer GPIO1.8 (Pin_8)
- net 3.3v: now reaches RPiGPIO1.1 (Pin_1)
- net 3.3v: now also GPIO1.8 (Pin_8)
- net VCC renamed 5v
- no-connect marks 10 -> 9

Commit message: version 7
Parts:
- added J1: Conn_01x01, Custom:raspberrypi_2_3, symbol Connector_Generic:Conn_01x01
- added J2: 1x02, Custom:JST_PH_S2B-PH-K_1x02_P2.00mm_Horizontal, symbol Connector_Generic:Conn_01x02
- added SCD30: Conn_01x04_Socket, Custom:STEMMA QT 1x04, symbol Connector_Generic:Conn_01x04
- GPIO1: value 02x05 -> 02x03; footprint Connector_PinHeader_2.54mm:PinHeader_2x05_P2.54mm_Horizontal -> Custom:GPIO Header; symbol Connector_Generic:Conn_02x05_Odd_Even -> Connector_Generic:Conn_02x03_Odd_Even
- HUB1: footprint Connector_IDC:IDC-Header_2x08_P2.54mm_Horizontal -> Custom:HUB75
- IO1: footprint Connector_IDC:IDC-Header_2x03_P2.54mm_Horizontal -> Custom:JST_SH_SM06B-SRSS-TB_1x06-1MP_P1.00mm_Horizontal
- RPiGPIO1: footprint Connector_PinSocket_2.54mm:PinSocket_2x20_P2.54mm_Vertical -> Custom:RPi GPIO
Connections:
- net 5v: now also GPIO1.4 (Pin_4), J2.1 (Pin_1), SCD30.2 (Pin_2); no longer GPIO1.6 (Pin_6)
- net GPIO 13: now also GPIO1.1 (Pin_1); no longer GPIO1.5 (Pin_5)
- net GPIO 19: now also GPIO1.3 (Pin_3); no longer GPIO1.7 (Pin_7)
- net GPIO 2: now also SCD30.3 (Pin_3); no longer GPIO1.1 (Pin_1)
- net GPIO 26: now also GPIO1.5 (Pin_5); no longer GPIO1.2 (Pin_2)
- net GPIO 3: now also SCD30.4 (Pin_4); no longer GPIO1.3 (Pin_3)
- net GPIO 6: now also GPIO1.2 (Pin_2); no longer GPIO1.4 (Pin_4)
- net at BZ1.2 (+), HUB1.14 (Pin_14), HUB1.4 (Pin_4)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: now also GPIO1.6 (Pin_6), J2.2 (Pin_2), SCD30.1 (Pin_1); no longer GPIO1.10 (Pin_10), GPIO1.9 (Pin_9)
- net 3.3v: no longer names the net of RPiGPIO1.1 (Pin_1)
- net 3.3v: no longer GPIO1.8 (Pin_8)
- no-connect marks 9 -> 11
